File: JLC4_RoboChalangeBoards.kicad_pcb (KiCad board)
At the start: 2 copper layers, 102 x 102 mm, 209 parts, among them J1 BAT, J1 Conn_01x06_Pin, J1 Conn_01x08_Pin, J1 Conn_01x10_Pin, J1 USB, J1 USB_C_Receptacle_PowerOnly_6P, J10 Conn_01x04_Pin, J2 Bat+, J2 Conn_01x05, J2 Conn_01x08_Pin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

Commit message: r
Parts:
- added G***: LOGO, LOGO, B.Cu at (117.0, 121.8)
